File: garbox.kicad_pcb (KiCad board)
At the start: 4 copper layers, 58.4 x 65.3 mm, 79 parts, among them J1 Batteries Terminal, J2 Speaker Terminals, J3 USB4056-03-A_REVA2, J4 MSD-4-A, U1 ESP32-S3-WROOM-1-N4R8, U10 FT231XQ-T, U2 CS4344-CZZR, U3 PAM8302AASCR, U4 AMS1117-3.3, U5 AMS1117-5.0, U6 BQ25887RGER, U7 CPDQ5V0-HF, U8 CPDQ5V0-HF, U9 CPDQ5V0-HF

Commit message: meant to put these in the last commit
Parts:
- added J5: SD_Header, TS_110_G_A:SAMTEC_TS-110-G-A, F.Cu at (163.5, 111.3)
- added J6: PowerBreakoutHeader, TS_110_G_A:SAMTEC_TS-110-G-A, F.Cu at (113.5, 75.2)
- added J7: BMS_Header, TS_110_G_A:SAMTEC_TS-110-G-A, F.Cu at (113.8, 45.2)
- added J8: Audio_Header, TS_110_G_A:SAMTEC_TS-110-G-A, F.Cu at (174.5, 48.0)
- added J9: GPIO_Header, TS_110_G_A:SAMTEC_TS-110-G-A, F.Cu at (174.8, 77.5)
- added R30: 22, Resistor_SMD:R_0201_0603Metric, F.Cu at (123.6, 48.8)
- added R31: 22, Resistor_SMD:R_0201_0603Metric, F.Cu at (123.6, 50.5)
- J2: value Speaker Terminals -> USB_Header; footprint TerminalBlock_MetzConnect:TerminalBlock_MetzConnect_Type011_RT05502HBLC_1x02_P5.00mm_Horizontal -> TS_110_G_A:SAMTEC_TS-110-G-A
- moved C29 181.6 mm to (235.6, 138.2), turned to 0 degrees
- moved C10 179.4 mm to (236.4, 135.3), turned to 0 degrees
- moved C8 177.0 mm to (236.4, 132.0), turned to 0 degrees
- moved C13 174.5 mm to (239.0, 138.0)
- moved C6 172.7 mm to (230.4, 135.9), turned to 0 degrees
- moved C31 171.1 mm to (236.8, 128.0)
- moved L1 167.9 mm to (230.9, 132.4)
- moved C4 166.8 mm to (236.8, 125.1)
- moved U6 166.6 mm to (231.4, 127.0), turned to 0 degrees
- moved R6 166.0 mm to (227.0, 131.5), turned to 0 degrees
- moved R5 164.5 mm to (227.0, 129.8), turned to 0 degrees
- moved C27 159.3 mm to (106.0, 236.9), turned to 0 degrees
- moved R21 158.6 mm to (227.0, 133.3), turned to 0 degrees
- moved R4 158.0 mm to (227.0, 128.0), turned to 0 degrees
- moved R3 156.9 mm to (227.0, 126.3), turned to 0 degrees
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Connections:
- net /Audio/AMP_ENABLE renamed /AMP_ENABLE
- net /Audio/i2s_LRCK renamed /i2s_LRCK
- net /Audio/i2s_MCLK renamed /i2s_MCLK
- net /Audio/i2s_SCLK renamed /i2s_SCLK
- net /Audio/i2s_SDIN renamed /i2s_SDIN
- net /BatteryManagement/BMS_Interrupt renamed /BMS_Interrupt
- net /BatteryManagement/ChargeStatus renamed /ChargeStatus
- net /BatteryManagement/PSEL renamed /PSEL
- net /BatteryManagement/PowerGood renamed /PowerGood
- net /BatteryManagement/SCL renamed /SCL
- net /BatteryManagement/SDA renamed /SDA
- C11 pad 2: /BatteryManagement/PowerIn -> /USB_PowerSupply
- C13 pad 1: /BatteryManagement/PowerIn -> /USB_PowerSupply
- C17 pad 2: /BatteryManagement/PowerIn -> /USB_PowerSupply
- C2 pad 2: +3.3V -> /PowerRegulation/3V3
- C22 pad 1: /Audio/Spk- -> /Spk-
- C23 pad 1: /Audio/Spk+ -> /Spk+
- C4 pad 1: /BatteryManagement/PowerIn -> /USB_PowerSupply
- C5 pad 2: +5V -> /PowerRegulation/5V
- FB2 pad 1: /Audio/Spk- -> /Spk-
- FB3 pad 1: /Audio/Spk+ -> /Spk+
- J3 pad A4: /BatteryManagement/PowerIn -> /USB_PowerSupply
- J3 pad A9: /BatteryManagement/PowerIn -> /USB_PowerSupply
- J3 pad B4: /BatteryManagement/PowerIn -> /USB_PowerSupply
- J3 pad B9: /BatteryManagement/PowerIn -> /USB_PowerSupply
- R15 pad 1: /USB_Data&Power/FLASH_RXD -> /FLASH_RXD
- R16 pad 1: /USB_Data&Power/FLASH_TXD -> /FLASH_TXD
- R20 pad 2: /USB_Data&Power/CTS# -> /CTS#
- R23 pad 1: Net-(U1-IO19) -> /GPLED_01
- R8 pad 1: Net-(U1-IO20) -> /GPLED_02
- U1 pad 10: unconnected-(U1-IO17-Pad10) -> /GPLED_01
- U1 pad 11: unconnected-(U1-IO18-Pad11) -> /GPLED_02
- U1 pad 12: unconnected-(U1-IO8-Pad12) -> /GPIO_08
- U1 pad 15: unconnected-(U1-IO3-Pad15) -> /GPIO_03
- U1 pad 16: unconnected-(U1-IO46-Pad16) -> /GPIO_46
- U1 pad 17: unconnected-(U1-IO9-Pad17) -> /GPIO_09
- U1 pad 25: unconnected-(U1-IO48-Pad25) -> /GPIO_48
- U1 pad 27: /USB_Data&Power/DTR# -> /FLASH_TXD
- U1 pad 3: /USB_Data&Power/RTS# -> /RTS#
- U1 pad 32: unconnected-(U1-IO39-Pad32) -> /GPIO_39
- U1 pad 33: /USB_Data&Power/CTS# -> /DTR#
- U1 pad 34: unconnected-(U1-IO41-Pad34) -> /GPIO_41
- U1 pad 35: unconnected-(U1-IO42-Pad35) -> /GPIO_42
- U1 pad 38: unconnected-(U1-IO2-Pad38) -> /GPIO_02
- U1 pad 39: unconnected-(U1-IO1-Pad39) -> /GPIO_01
- U10 pad 1: /USB_Data&Power/FLASH_RXD -> /FLASH_RXD
- U10 pad 12: /BatteryManagement/PowerIn -> /USB_PowerSupply
- U10 pad 17: /USB_Data&Power/FLASH_TXD -> /FLASH_TXD
- U10 pad 18: /USB_Data&Power/DTR# -> /DTR#
- U10 pad 19: /USB_Data&Power/RTS# -> /RTS#
- U10 pad 6: /USB_Data&Power/CTS# -> /CTS#
- U4 pad 2: +3.3V -> /PowerRegulation/3V3
- U5 pad 2: +5V -> /PowerRegulation/5V
- U6 pad 23: /BatteryManagement/PowerIn -> /USB_PowerSupply
- U9 pad 1: /BatteryManagement/PowerIn -> /USB_PowerSupply
Routing:
- net +5V: track 82.5 -> 0.00 mm, vias 7 -> 0
- net GND: track 49.0 -> 0.00 mm, vias 45 -> 0
- net /USB_Data&Power/CTS#: track 36.4 -> 0.00 mm, vias 4 -> 0
- net /BatteryManagement/PowerIn: track 34.3 -> 0.00 mm, vias 4 -> 0
- net /USB_Data&Power/FLASH_TXD: track 34.2 -> 0.00 mm, vias 2 -> 0
- net /USB_Data&Power/RTS#: track 34.0 -> 0.00 mm, vias 2 -> 0
- net /i2s_SDIN: track 33.4 -> 0.00 mm, vias 2 -> 0
- net /USB_Data&Power/DTR#: track 33.3 -> 0.00 mm, vias 2 -> 0
- net /USB_Data&Power/FLASH_RXD: track 31.9 -> 0.00 mm, vias 2 -> 0
- net /i2s_SCLK: track 31.0 -> 0.00 mm, vias 2 -> 0
- net /i2s_LRCK: track 28.8 -> 0.00 mm, vias 2 -> 0
- net Net-(U10-3V3OUT): track 27.6 -> 0.00 mm, vias 2 -> 0
- net /i2s_MCLK: track 25.9 -> 0.00 mm, vias 2 -> 0
- net /AMP_ENABLE: track 25.7 -> 0.00 mm, vias 2 -> 0
- net /BatteryManagement/PackMid: track 20.9 -> 0.00 mm, vias 1 -> 0
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- removed copper zone on F.Cu, net +3.3V
- removed copper zone on In2.Cu, net +3.3V
- removed copper zone on F.Cu, net +5V
- removed copper zone on F.Cu, net /BatteryManagement/PackMid
- removed copper zone on F.Cu, net /BatteryManagement/PackPlus
- removed copper zone on F.Cu, net /BatteryManagement/PowerIn
- removed copper zone on In2.Cu, net /BatteryManagement/PowerIn
- removed copper zone on In1.Cu, net GND
- removed copper zone on F.Cu, net Net-(C29-Pad1)
- removed copper zone on F.Cu, net Net-(C31-Pad2)
- removed copper zone on F.Cu, net Net-(C8-Pad1)
- removed copper zone on F.Cu, net Net-(J3-SHELL_GND)
- removed copper zone on In1.Cu, net Net-(J3-SHELL_GND)
- removed copper zone on F.Cu, net Net-(U10-3V3OUT)
Other:
- board size 58.4 x 65.3 mm -> 78.7 x 147.3 mm

Commit message: Finished preliminary routing of v1.1 of the board
Parts:
- added C24: 10uF, CL31A106KBHNNNE:CAP_CL31_SAM, F.Cu at (120.9, 100.3)
- moved R6 144.8 mm to (88.3, 90.2), turned to 90 degrees
- moved R5 142.4 mm to (90.2, 90.2), turned to 90 degrees
- moved C29 141.3 mm to (99.1, 101.6)
- moved R4 140.1 mm to (88.9, 104.1), turned to 180 degrees
- moved R21 139.1 mm to (88.9, 116.8), turned to 180 degrees
- moved C10 138.9 mm to (102.2, 99.1)
- moved R3 138.8 mm to (88.9, 111.8), turned to 180 degrees
- moved C8 138.6 mm to (100.3, 105.4), turned to 90 degrees
- moved R2 138.5 mm to (88.9, 114.3), turned to 180 degrees
- moved C31 136.8 mm to (101.0, 111.1), turned to -90 degrees
- moved C15 136.4 mm to (129.2, 100.3)
- moved L1 134.9 mm to (97.8, 110.5), turned to -90 degrees
- moved C13 132.9 mm to (108.6, 112.4)
- moved C7 131.3 mm to (121.3, 105.4), turned to -90 degrees
- moved U2 130.1 mm to (129.2, 103.5), turned to 180 degrees
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Connections:
- C7 pad 1: /Audio/A_OUT_R -> /PostDac
- J2 pad 01: /USB_Data&Power/DSR# -> /USB_Data&Power/USB_D-
- J2 pad 02: /USB_Data&Power/DCD# -> /USB_Data&Power/USB_D+
- J2 pad 03: /USB_Data&Power/USB_D- -> /USB_PowerSupply
- J2 pad 04: /USB_Data&Power/USB_D+ -> /FLASH_TXD
- J2 pad 05: /FLASH_TXD -> /DTR#
- J2 pad 06: /DTR# -> /RTS#
- J2 pad 07: /FLASH_TXD -> /FLASH_RXD
- J2 pad 08: /FLASH_RXD -> /USB_Data&Power/DSR#
- J2 pad 09: /RTS# -> /USB_Data&Power/DCD#
- J2 pad 10: /USB_PowerSupply -> /CTS#
- J5 pad 02: GND -> /SD_DAT2
- J5 pad 03: /SD_DAT2 -> /SD_DAT3
- J5 pad 04: /SD_DAT3 -> /SD_CMD
- J5 pad 05: /SD_CMD -> +3.3V
- J5 pad 06: /SD_CLK -> GND
- J5 pad 07: /SD_DAT0 -> /SD_CLK
- J5 pad 08: /SD_DAT1 -> /SD_DAT0
- J5 pad 09: /SD_CD -> /SD_DAT1
- J5 pad 10: +3.3V -> /SD_CD
- J7 pad 01: /USB_OTG_D+ -> GND
- J7 pad 02: /USB_OTG_D- -> GND
- J7 pad 03: GND -> /PSEL
- J7 pad 04: GND -> /PowerGood
- J7 pad 05: /BMS_Interrupt -> /ChargeStatus
- J7 pad 06: /PSEL -> /SDA
- J7 pad 07: /PowerGood -> /SCL
- J7 pad 08: /ChargeStatus -> /BMS_Interrupt
- J7 pad 09: /SDA -> /USB_OTG_D+
- J7 pad 10: /SCL -> /USB_OTG_D-
- J8 pad 01: GND -> /i2s_MCLK
- J8 pad 02: /Spk- -> /i2s_LRCK
- J8 pad 03: GND -> /i2s_SCLK
- J8 pad 04: /Spk+ -> /i2s_SDIN
- J8 pad 05: GND -> /PostDac
- J8 pad 06: /AMP_ENABLE -> /PreAmp
- J8 pad 07: /i2s_MCLK -> /AMP_ENABLE
- J8 pad 08: /i2s_LRCK -> /Spk-
- J8 pad 09: /i2s_SCLK -> GND
- J8 pad 10: /i2s_SDIN -> /Spk+
- J9 pad 01: /GPIO_08 -> /GPIO_03
- J9 pad 02: /GPIO_03 -> /GPIO_46
- J9 pad 03: /GPIO_46 -> /GPIO_09
- J9 pad 04: /GPIO_09 -> /GPIO_17
- J9 pad 05: /GPIO_48 -> /GPIO_16
- J9 pad 06: /GPIO_39 -> /GPIO_15
- J9 pad 07: /GPIO_41 -> /GPIO_07
- J9 pad 08: /GPIO_42 -> /GPIO_06
- J9 pad 09: /GPIO_02 -> /GPIO_05
- J9 pad 10: /GPIO_01 -> /GPIO_08
- R22 pad 2: /Audio/IN+ -> /PreAmp
- R24 pad 1: /Audio/IN+ -> /PreAmp
- U1 pad 10: /GPLED_01 -> /GPIO_17
- U1 pad 12: /GPIO_08 -> /GPLED_01
- U1 pad 18: /SD_CD -> /BMS_Interrupt
- U1 pad 19: /SD_DAT1 -> /SCL
- U1 pad 20: /SD_DAT0 -> /SDA
- U1 pad 21: /SD_CLK -> /ChargeStatus
- U1 pad 22: /SD_CMD -> /PowerGood
- U1 pad 23: /SD_DAT3 -> /PSEL
- U1 pad 24: /SD_DAT2 -> /i2s_MCLK
- U1 pad 25: /GPIO_48 -> /i2s_LRCK
- U1 pad 26: /AMP_ENABLE -> /i2s_SCLK
- U1 pad 27: /FLASH_TXD -> /DTR#
- U1 pad 28: /i2s_MCLK -> /i2s_SDIN
- U1 pad 29: /i2s_LRCK -> /AMP_ENABLE
- U1 pad 30: /i2s_SCLK -> /SD_CD
- U1 pad 31: /i2s_SDIN -> /SD_DAT1
- U1 pad 32: /GPIO_39 -> /SD_DAT0
- U1 pad 33: /DTR# -> /CTS#
- U1 pad 34: /GPIO_41 -> /SD_CLK
- U1 pad 35: /GPIO_42 -> /SD_CMD
- U1 pad 38: /GPIO_02 -> /SD_DAT3
- U1 pad 39: /GPIO_01 -> /SD_DAT2
- U1 pad 4: /BMS_Interrupt -> /GPIO_08
- U1 pad 5: /SCL -> /GPIO_05
- U1 pad 6: /SDA -> /GPIO_06
- U1 pad 7: /ChargeStatus -> /GPIO_07
- U1 pad 8: /PowerGood -> /GPIO_15
- U1 pad 9: /PSEL -> /GPIO_16
- U2 pad 10: /Audio/A_OUT_R -> /PostDac
- U3 pad 3: /Audio/IN+ -> /PreAmp
Routing:
- net /CTS#: track 0.00 -> 149.2 mm, vias 0 -> 3
- net /FLASH_RXD: track 0.00 -> 140.7 mm, vias 0 -> 3
- net /FLASH_TXD: track 0.00 -> 138.2 mm, vias 0 -> 2
- net /SD_DAT1: track 6.70 -> 131.4 mm, vias 0 -> 1
- net /SD_DAT2: track 5.39 -> 128.5 mm, vias 0 -> 1
- net /SD_DAT0: track 5.36 -> 128.2 mm, vias 0 -> 1
- net /SD_CD: track 0.00 -> 122.6 mm, vias 0 -> 1
- net /SD_DAT3: track 6.67 -> 129.0 mm, vias 0 -> 1
- net /SD_CMD: track 5.34 -> 127.0 mm, vias 0 -> 1
- net /SD_CLK: track 0.00 -> 121.6 mm, vias 0 -> 2
- net /RTS#: track 0.00 -> 116.2 mm, vias 0 -> 2
- net /DTR#: track 0.00 -> 113.7 mm, vias 0 -> 1
- net GND: track 0.00 -> 106.8 mm, vias 0 -> 46
- net /AMP_ENABLE: track 0.00 -> 106.6 mm
- net +5V: track 0.00 -> 95.2 mm, vias 0 -> 2
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- added copper zone on In2.Cu, net +3.3V
- added copper zone on F.Cu, net +5V
- added copper zone on F.Cu, net /BatteryManagement/PackPlus
- added copper zone on F.Cu, net /PowerRegulation/3V3
- added copper zone on F.Cu, net /PowerRegulation/5V
- added copper zone on F.Cu, net /USB_PowerSupply
- added copper zone on In2.Cu, net /USB_PowerSupply
- added copper zone on In1.Cu, net GND
- added copper zone on F.Cu, net Net-(J3-SHELL_GND)
Other:
- outline, holes or cut-outs redrawn
- board text added: "18650 for reference"
- board text added: "3V3"
- board text added: "5V"
- board text added: "AMP_ENABLE"
- board text added: "AUDIO"
- board text added: "BMS"
- board text added: "BMS_Interrupt"
- board text added: "CTS#"
- board text added: "ChargeStatus"
- board text added: "DCD#"
- board text added: "DSR#"
- board text added: "DTR#"
- board text added: "FLASH_RXD"
- board text added: "FLASH_TXD"
- board text added: "GND"
- board text added: "GPIO"
- board text added: "LED1 GPIO 08"
- board text added: "LED2 GPIO 18"
- board text added: "POWER"
- board text added: "PSEL"
- board text added: "Post-DAC Sig."
- board text added: "PowerGood"
- board text added: "Pre-Amp Sig."
- board text added: "RTS#"
- board text added: "SCL"
- board text added: "SD/MMC"
- board text added: "SDA"
- board text added: "SD_CD"
- board text added: "SD_CLK"
- board text added: "SD_CMD"
- board text added: "SD_DAT0"
- board text added: "SD_DAT1"
- board text added: "SD_DAT2"
- board text added: "SD_DAT3"
- board text added: "SPK+"
- board text added: "SPK-"
- board text added: "USB/UART"
- board text added: "USB_D+"
- board text added: "USB_D-"
- board text added: "USB_OTG_D+"
- board text added: "USB_OTG_D-"
- board text added: "i"
- board text added: "i2s_LRCK"
- board text added: "i2s_MCLK"
- board text added: "i2s_SCLK"
- board text added: "i2s_SDIN"
- board text added: "o"

Commit message: Cleaned up silkscreen and finished routing
Routing:
- net GND: track 106.8 -> 108.3 mm, vias 46 -> 47
Other:
- board text added: "Calories 0"
- board text added: "Cholesterol 0mg 0%"
- board text added: "Copper 28g ???%"
- board text added: "Fiber 14g 50%"
- board text added: "GPIO_03"
- board text added: "GPIO_05"
- board text added: "GPIO_06"
- board text added: "GPIO_07"
- board text added: "GPIO_08"
- board text added: "GPIO_09"
- board text added: "GPIO_15"
- board text added: "GPIO_16"
- board text added: "GPIO_17"
- board text added: "GPIO_46"
- board text added: "Lead 2g 999%"
- board text added: "Nutrition Facts"
- board text added: "Per serving %DV"
- board text added: "Protein 0g"
- board text added: "Serving size 1 PCB (44g)"
- board text added: "Sodium 0mg 0%"
- board text added: "Total Fat 0g 0%"
- board text added: "garbox v1.1 K.Q. 08/2025"

Commit message: fixed incorrect gpio and added silkscreen funny
Parts:
- moved D1 17.9 mm to (85.0, 139.0), turned to 180 degrees
- moved D2 17.9 mm to (80.3, 139.0), turned to 180 degrees
- moved R12 14.5 mm to (91.0, 151.7), turned to 180 degrees
- moved R11 13.0 mm to (91.0, 149.0), turned to 180 degrees
- moved D3 11.6 mm to (98.0, 48.7), turned to -90 degrees
- moved D4 4.73 mm to (93.0, 48.7), turned to -90 degrees
Connections:
- net /GPIO_08 renamed /GPIO_04
Routing:
- net Net-(D2-A): track 1.90 -> 17.1 mm
- net Net-(D3-A): track 21.1 -> 7.51 mm
- net Net-(D1-A): track 1.90 -> 12.5 mm
- net Net-(U10-3V3OUT): track 45.2 -> 36.3 mm
- net /USB_Data&Power/CBUS1: track 34.1 -> 38.0 mm
- net Net-(D4-A): track 17.7 -> 14.0 mm
- net /USB_Data&Power/CBUS2: track 21.7 -> 25.1 mm
- net GND: track 108.3 -> 109.4 mm
Other:
- outline, holes or cut-outs redrawn
- board text added: "GPIO_04"
- board text added: "LED1 GPIO_08"
- board text added: "LED2 GPIO_18"
- board text added: "USB_POWER"
- board text removed: "GPIO_08"
- board text removed: "LED1 GPIO 08"
- board text removed: "LED2 GPIO 18"
