File: audio.kicad_sch (KiCad schematic)
At the start: 14 parts, among them U2 CS4344-CZZR, U3 PAM8302AASCR

Commit message: Finished preliminary routing of v1.1 of the board
Parts:
- added C24: 10uF, CL31A106KBHNNNE:CAP_CL31_SAM, symbol CL31A106KBHNNNE:CL31A106KBHNNNE
Connections:
- net +5V: now also C24.2
- net GND: now also C24.1
- net A_OUT_R renamed PostDAC
- net IN+ renamed PreAmp
Other:
- note added: "Header breakout"
Changed lines of the file:
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@@
+		)
+	)
+	(rectangle
+		(start 27.94 78.74)
+		(end 53.34 91.44)
+		(stroke
+			(width 0)
+			(type default)
+		)
+		(fill
+			(type none)
 		)
 	)
@@
 				(thickness 0.254)
 				(bold yes)
+			)
+		)
+	)
+	(text "Header breakout"
+		(exclude_from_sim no)
+		(at 34.036 79.756 0)
+		(effects
+			(font
+				(size 0.889 0.889)
 			)
 		)
@@
 	)
 	(junction
+		(at 170.18 57.15)
+		(diameter 0)
+		(color 0 0 0 0)
+	)
+	(junction
 		(at 148.59 97.79)
 		(diameter 0)
@@
 	)
 	(junction
+		(at 171.45 54.61)
+		(diameter 0)
+		(color 0 0 0 0)
+	)
+	(junction
 		(at 90.17 77.47)
 		(diameter 0)
@@
 	(wire
 		(pts
+			(xy 179.07 49.53) (xy 179.07 54.61)
+		)
+		(stroke
+			(width 0)
+			(type default)
+		)
+	)
+	(wire
+		(pts
 			(xy 90.17 67.31) (xy 95.25 67.31)
 		)
@@
 	(wire
 		(pts
+			(xy 186.69 52.07) (xy 186.69 49.53)
+		)
+		(stroke
+			(width 0)
+			(type default)
+		)
+	)
+	(wire
+		(pts
 			(xy 106.68 87.63) (xy 115.57 87.63)
 		)
@@
 	(wire
 		(pts
+			(xy 43.18 88.9) (xy 39.37 88.9)
+		)
+		(stroke
+			(width 0)
+			(type default)
+		)
+	)
+	(wire
+		(pts
+			(xy 186.69 62.23) (xy 179.07 62.23)
+		)
+		(stroke
+			(width 0)
+			(type default)
+		)
+	)
+	(wire
+		(pts
 			(xy 148.59 97.79) (xy 148.59 93.98)
 		)
@@
 	(wire
 		(pts
+			(xy 186.69 49.53) (xy 179.07 49.53)
+		)
+		(stroke
+			(width 0)
+			(type default)
+		)
+	)
+	(wire
+		(pts
+			(xy 186.69 59.69) (xy 186.69 62.23)
+		)
+		(stroke
+			(width 0)
+			(type default)
+		)
+	)
+	(wire
+		(pts
+			(xy 179.07 62.23) (xy 179.07 57.15)
+		)
+		(stroke
+			(width 0)
+			(type default)
+		)
+	)
+	(wire
+		(pts
 			(xy 161.29 109.22) (xy 161.29 107.95)
 		)
@@
 	(wire
 		(pts
+			(xy 171.45 54.61) (xy 179.07 54.61)
+		)
+		(stroke
+			(width 0)
+			(type default)
+		)
+	)
+	(wire
+		(pts
 			(xy 95.25 76.2) (xy 95.25 77.47)
 		)
@@
 	(wire
 		(pts
+			(xy 179.07 57.15) (xy 170.18 57.15)
+		)
+		(stroke
+			(width 0)
+			(type default)
+		)
+	)
+	(wire
+		(pts
 			(xy 100.33 121.92) (xy 104.14 121.92)
 		)
@@
 	(wire
 		(pts
+			(xy 43.18 85.09) (xy 39.37 85.09)
+		)
+		(stroke
+			(width 0)
+			(type default)
+		)
+	)
+	(wire
+		(pts
 			(xy 95.25 67.31) (xy 95.25 68.58)
 		)
@@
 			(width 0)
 			(type default)
+		)
+	)
+	(label "A_OUT_R"
+		(at 43.18 88.9 0)
+		(effects
+			(font
+				(size 1.27 1.27)
+			)
+			(justify left bottom)
 		)
 	)
 	(label "IN+"
 		(at 100.33 121.92 0)
+		(effects
+			(font
+				(size 1.27 1.27)
+			)
+			(justify left bottom)
+		)
+	)
+	(label "IN+"
+		(at 43.18 85.09 0)
 		(effects
 			(font
@@
 		)
 	)
+	(hierarchical_label "PreAmp"
+		(shape passive)
+		(at 39.37 85.09 180)
+		(effects
+			(font
+				(size 1.27 1.27)
+			)
+			(justify right)
+		)
+	)
 	(hierarchical_label "AMP_ENABLE"
 		(shape input)
@@
 		(shape input)
 		(at 88.9 59.69 180)
+		(effects
+			(font
+				(size 1.27 1.27)
+			)
+			(justify right)
+		)
+	)
+	(hierarchical_label "PostDAC"
+		(shape passive)
+		(at 39.37 88.9 180)
 		(effects
 			(font
@@
 					(unit 1)
 				)
+			)
+		)
+	)
+	(symbol
+		(lib_id "CL31A106KBHNNNE:CL31A106KBHNNNE")
+		(at 186.69 59.69 90)
+		(unit 1)
+		(exclude_from_sim no)
+		(in_bom yes)
+		(on_board yes)
+		(dnp no)
+		(property "Reference" "C24"
+			(at 188.722 55.118 90)
+			(effects
+				(font
+					(size 1.524 1.524)
+				)
+				(justify right)
+			)
+		)
+		(property "Value" "10uF"
+			(at 187.452 57.658 90)
+			(effects
+				(font
+					(size 1.524 1.524)
+				)
+				(justify right)
+			)
+		)
+		(property "Footprint" "CL31A106KBHNNNE:CAP_CL31_SAM"
+			(at 186.69 59.69 0)
+			(effects
+				(font
+					(size 1.27 1.27)
+					(italic yes)
+				)
+				(hide yes)
+			)
+		)
+		(property "Datasheet" "CL31A106KBHNNNE"
+			(at 186.69 59.69 0)
+			(effects
+				(font
+					(size 1.27 1.27)
+					(italic yes)
+				)
+				(hide yes)
+			)
+		)
+		(property "Description" "CL31A106KBHNNNE"
+			(at 186.69 59.69 0)
+			(effects
+				(font
+					(size 1.27 1.27)
+				)
+				(hide yes)
+			)
+		)
+		(pin "2"
+		)
+		(pin "1"
+		)
+		(instances
+			(project "garbox"
+				(path "/e66b6024-0366-4f6a-a697-473ffced0d7c/7a530924-455b-4752-9a2b-034dacbf5709"
+					(reference "C24")
+					(unit 1)
+				)

Commit message: designated MPN parts from JLC library
Parts:
- C15: MPN (none) -> C1525
- C16, C20, C24, C9: MPN (none) -> C13585
- C22, C23: MPN (none) -> C1603
- C27: MPN (none) -> C1848
- C7: MPN (none) -> C51412
- FB2, FB3: MPN (none) -> C1002
- R22: MPN (none) -> C23179
- R24: MPN (none) -> C25804
- U2: MPN (none) -> C2895053
- U3: MPN (none) -> C113367
Changed lines of the file:
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@@
+			)
+		)
+		(property "MPN" "C1603"
+			(at 163.83 130.81 0)
+			(effects
+				(font
+					(size 1.27 1.27)
+				)
+				(hide yes)
 			)
 		)
@@
 			)
 		)
+		(property "MPN" "C1848"
+			(at 165.1 104.14 90)
+			(effects
+				(font
+					(size 1.27 1.27)
+				)
+				(hide yes)
+			)
+		)
 		(pin "2"
 		)
@@
 			)
 		)
+		(property "MPN" "C1603"
+			(at 176.53 130.81 0)
+			(effects
+				(font
+					(size 1.27 1.27)
+				)
+				(hide yes)
+			)
+		)
 		(pin "2"
 		)
@@
 		(property "Description" "Ferrite bead"
 			(at 156.21 124.46 0)
+			(effects
+				(font
+					(size 1.27 1.27)
+				)
+				(hide yes)
+			)
+		)
+		(property "MPN" "C1002"
+			(at 156.21 124.46 90)
 			(effects
 				(font
@@
 			)
 		)
+		(property "MPN" "C2895053"
+			(at 90.17 52.07 0)
+			(effects
+				(font
+					(size 1.27 1.27)
+				)
+				(hide yes)
+			)
+		)
 		(pin "6"
 		)
@@
 			)
 		)
+		(property "MPN" "C13585"
+			(at 90.17 77.47 0)
+			(effects
+				(font
+					(size 1.27 1.27)
+				)
+				(hide yes)
+			)
+		)
 		(pin "2"
 		)
@@
 		(property "Description" "Ferrite bead"
 			(at 156.21 116.84 0)
+			(effects
+				(font
+					(size 1.27 1.27)
+				)
+				(hide yes)
+			)
+		)
+		(property "MPN" "C1002"
+			(at 156.21 116.84 90)
 			(effects
 				(font
@@
 			)
 		)
+		(property "MPN" "C13585"
+			(at 157.48 106.68 90)
+			(effects
+				(font
+					(size 1.27 1.27)
+				)
+				(hide yes)
+			)
+		)
 		(pin "2"
 		)
@@
 			)
 		)
+		(property "MPN" "C13585"
+			(at 186.69 59.69 90)
+			(effects
+				(font
+					(size 1.27 1.27)
+				)
+				(hide yes)
+			)
+		)
 		(pin "2"
 		)
@@
 		(property "Description" "0603WAF4700T5E"
 			(at 132.842 77.216 0)
+			(effects
+				(font
+					(size 1.27 1.27)
+				)
+				(hide yes)
+			)
+		)
+		(property "MPN" "C23179"
+			(at 129.54 87.63 0)
 			(effects
 				(font
@@
 			)
 		)
+		(property "MPN" "C51412"
+			(at 118.11 87.63 0)
+			(effects
+				(font
+					(size 1.27 1.27)
+				)
+				(hide yes)
+			)
+		)
 		(pin "1"
 		)
@@
 			)
 		)
+		(property "MPN" "C1525"
+			(at 95.25 76.2 0)
+			(effects
+				(font
+					(size 1.27 1.27)
+				)
+				(hide yes)
+			)
+		)
 		(pin "2"
 		)
@@
 			)
 		)
+		(property "MPN" "C25804"
+			(at 135.89 93.98 90)
+			(effects
+				(font
+					(size 1.27 1.27)
+				)
+				(hide yes)
+			)
+		)
 		(pin "2"
 		)
@@
 			)
 		)
+		(property "MPN" "C113367"
+			(at 104.14 116.84 0)
+			(effects
+				(font
+					(size 1.27 1.27)
+				)
+				(hide yes)
+			)
+		)
 		(pin "8"
 		)
@@
 			(effects
 				(font
+					(size 1.27 1.27)
+				)
+				(hide yes)
+			)
+		)
+		(property "MPN" "C13585"
+			(at 161.29 76.2 90)
+			(effects
+				(font

Commit message: Updated part numbers
Parts:
- C16: footprint Capacitor_SMD:C_0201_0603Metric -> CL31A106KBHNNNE:CAP_CL31_SAM
Changed lines of the file:
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@@
+			)
+		)
+		(property "FIX" ""
+			(at 163.83 130.81 0)
+			(effects
+				(font
+					(size 1.27 1.27)
+				)
+				(hide yes)
 			)
 		)
@@
 			)
 		)
+		(property "FIX" ""
+			(at 165.1 104.14 90)
+			(effects
+				(font
+					(size 1.27 1.27)
+				)
+				(hide yes)
+			)
+		)
 		(pin "2"
 		)
@@
 			)
 		)
+		(property "FIX" ""
+			(at 176.53 130.81 0)
+			(effects
+				(font
+					(size 1.27 1.27)
+				)
+				(hide yes)
+			)
+		)
 		(pin "2"
 		)
@@
 		)
 		(property "MPN" "C1002"
+			(at 156.21 124.46 90)
+			(effects
+				(font
+					(size 1.27 1.27)
+				)
+				(hide yes)
+			)
+		)
+		(property "FIX" ""
 			(at 156.21 124.46 90)
 			(effects
@@
 			)
 		)
+		(property "FIX" ""
+			(at 90.17 52.07 0)
+			(effects
+				(font
+					(size 1.27 1.27)
+				)
+				(hide yes)
+			)
+		)
 		(pin "6"
 		)
@@
 			)
 		)
-		(property "Footprint" "Capacitor_SMD:C_0201_0603Metric"
+		(property "Footprint" "CL31A106KBHNNNE:CAP_CL31_SAM"
 			(at 90.17 77.47 0)
 			(effects
@@
 			)
 		)
+		(property "FIX" ""
+			(at 90.17 77.47 0)
+			(effects
+				(font
+					(size 1.27 1.27)
+				)
+				(hide yes)
+			)
+		)
 		(pin "2"
 		)
@@
 		)
 		(property "MPN" "C1002"
+			(at 156.21 116.84 90)
+			(effects
+				(font
+					(size 1.27 1.27)
+				)
+				(hide yes)
+			)
+		)
+		(property "FIX" ""
 			(at 156.21 116.84 90)
 			(effects
@@
 			)
 		)
+		(property "FIX" ""
+			(at 157.48 106.68 90)
+			(effects
+				(font
+					(size 1.27 1.27)
+				)
+				(hide yes)
+			)
+		)
 		(pin "2"
 		)
@@
 			)
 		)
+		(property "FIX" ""
+			(at 186.69 59.69 90)
+			(effects
+				(font
+					(size 1.27 1.27)
+				)
+				(hide yes)
+			)
+		)
 		(pin "2"
 		)
@@
 		)
 		(property "MPN" "C23179"
+			(at 129.54 87.63 0)
+			(effects
+				(font
+					(size 1.27 1.27)
+				)
+				(hide yes)
+			)
+		)
+		(property "FIX" ""
 			(at 129.54 87.63 0)
 			(effects
@@
 			)
 		)
+		(property "FIX" ""
+			(at 118.11 87.63 0)
+			(effects
+				(font
+					(size 1.27 1.27)
+				)
+				(hide yes)
+			)
+		)
 		(pin "1"
 		)
@@
 			)
 		)
+		(property "FIX" ""
+			(at 95.25 76.2 0)
+			(effects
+				(font
+					(size 1.27 1.27)
+				)
+				(hide yes)
+			)
+		)
 		(pin "2"
 		)
@@
 			)
 		)
+		(property "FIX" ""
+			(at 135.89 93.98 90)
+			(effects
+				(font
+					(size 1.27 1.27)
+				)
+				(hide yes)
+			)
+		)
 		(pin "2"
 		)
@@
 			)
 		)
+		(property "FIX" ""
+			(at 104.14 116.84 0)
+			(effects
+				(font
+					(size 1.27 1.27)
+				)
+				(hide yes)
+			)
+		)
 		(pin "8"
 		)
@@
 			(at 161.29 76.2 90)
 			(effects
+				(font
+					(size 1.27 1.27)
+				)
+				(hide yes)
+			)
+		)
+		(property "FIX" ""
+			(at 161.29 76.2 90)
+			(effects
