File: battpack.kicad_sch (KiCad schematic)
At the start: 1 part, among them J1 Batteries Terminal

Commit message: designated MPN parts from JLC library
Parts:
- J1: now left out of the parts list
Changed lines of the file:
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@@
 		(unit 1)
 		(exclude_from_sim no)
-		(in_bom yes)
+		(in_bom no)
 		(on_board yes)
 		(dnp no)
@@
 			(at 111.76 81.28 0)
 			(effects
+				(font
+					(size 1.27 1.27)
+				)
+				(hide yes)
+			)
+		)
+		(property "MPN" ""
+			(at 111.76 81.28 0)
+			(effects
