File: bms.kicad_sch (KiCad schematic)
At the start: 15 parts, among them U6 BQ25887RGER

Commit message: designated MPN parts from JLC library
Parts:
- C10: MPN (none) -> C13585
- C13: MPN (none) -> C1525
- C29: MPN (none) -> C1622
- C31, C4: MPN (none) -> C15850
- C6: MPN (none) -> C1779
- C8: MPN (none) -> C96123
- L1: MPN (none) -> C439775
- R2, R21, R3, R4: MPN (none) -> C25804
- R5: MPN (none) -> C23025
- R6: footprint Resistor_SMD:R_0201_0603Metric -> Resistor_SMD:R_2512_6332Metric; MPN (none) -> C16861
- U6: MPN (none) -> C2761614
Changed lines of the file:
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@@
 			)
 		)
-		(property "Footprint" "Resistor_SMD:R_0201_0603Metric"
+		(property "Footprint" "Resistor_SMD:R_2512_6332Metric"
 			(at 175.26 89.408 90)
 			(effects
@@
 			)
 		)
-		(property "Description" "0603WAF100JT5E"
+		(property "Description" "25121WJ0100T4E"
 			(at 175.26 87.63 0)
+			(effects
+				(font
+					(size 1.27 1.27)
+				)
+				(hide yes)
+			)
+		)
+		(property "MPN" "C16861"
+			(at 175.26 87.63 90)
 			(effects
 				(font
@@
 			)
 		)
+		(property "MPN" "C1525"
+			(at 109.22 67.31 90)
+			(effects
+				(font
+					(size 1.27 1.27)
+				)
+				(hide yes)
+			)
+		)
 		(pin "2"
 		)
@@
 			)
 		)
+		(property "MPN" "C25804"
+			(at 170.18 58.42 0)
+			(effects
+				(font
+					(size 1.27 1.27)
+				)
+				(hide yes)
+			)
+		)
 		(pin "2"
 		)
@@
 		(property "Description" "CL21A106KAYNNNE"
 			(at 120.65 80.01 0)
+			(effects
+				(font
+					(size 1.27 1.27)
+				)
+				(hide yes)
+			)
+		)
+		(property "MPN" "C15850"
+			(at 120.65 80.01 90)
 			(effects
 				(font
@@
 			)
 		)
+		(property "MPN" "C2761614"
+			(at 168.91 64.77 0)
+			(effects
+				(font
+					(size 1.27 1.27)
+				)
+				(hide yes)
+			)
+		)
 		(pin "2"
 		)
@@
 			)
 		)
+		(property "MPN" "C25804"
+			(at 186.69 58.42 0)
+			(effects
+				(font
+					(size 1.27 1.27)
+				)
+				(hide yes)
+			)
+		)
 		(pin "2"
 		)
@@
 		(property "Description" "CL21A106KAYNNNE"
 			(at 114.3 67.31 0)
+			(effects
+				(font
+					(size 1.27 1.27)
+				)
+				(hide yes)
+			)
+		)
+		(property "MPN" "C15850"
+			(at 114.3 67.31 90)
 			(effects
 				(font
@@
 			)
 		)
+		(property "MPN" "C1622"
+			(at 143.51 107.95 0)
+			(effects
+				(font
+					(size 1.27 1.27)
+				)
+				(hide yes)
+			)
+		)
 		(pin "2"
 		)
@@
 			)
 		)
+		(property "MPN" "C25804"
+			(at 201.93 58.42 0)
+			(effects
+				(font
+					(size 1.27 1.27)
+				)
+				(hide yes)
+			)
+		)
 		(pin "2"
 		)
@@
 		)
 		(property "Description" "0603WAF1002T5E"
+			(at 123.19 59.69 0)
+			(effects
+				(font
+					(size 1.27 1.27)
+				)
+				(hide yes)
+			)
+		)
+		(property "MPN" "C25804"
 			(at 123.19 59.69 0)
 			(effects
@@
 			)
 		)
+		(property "MPN" "C1779"
+			(at 180.34 99.06 90)
+			(effects
+				(font
+					(size 1.27 1.27)
+				)
+				(hide yes)
+			)
+		)
 		(pin "1"
 		)
@@
 			)
 		)
+		(property "MPN" "C96123"
+			(at 120.65 87.63 90)
+			(effects
+				(font
+					(size 1.27 1.27)
+				)
+				(hide yes)
+			)
+		)
 		(pin "2"
 		)
@@
 			)
 		)
+		(property "MPN" "C439775"
+			(at 113.03 77.47 0)
+			(effects
+				(font
+					(size 1.27 1.27)
+				)
+				(hide yes)
+			)
+		)
 		(pin "1"
 		)
@@
 			)
 		)
+		(property "MPN" "C13585"
+			(at 116.84 101.6 0)
+			(effects
+				(font
+					(size 1.27 1.27)
+				)
+				(hide yes)
+			)
+		)
 		(pin "2"
 		)
@@
 			(effects
 				(font
+					(size 1.27 1.27)
+				)
+				(hide yes)
+			)
+		)
+		(property "MPN" "C23025"
+			(at 175.26 85.09 90)
+			(effects
+				(font
