File: power.kicad_sch (KiCad schematic)
At the start: 6 parts, among them U4 AMS1117-3.3, U5 AMS1117-5.0

Commit message: designated MPN parts from JLC library
Parts:
- C1, C2, C3, C5: MPN (none) -> C13585
- U4: MPN (none) -> C6186
- U5: MPN (none) -> C6187
Changed lines of the file:
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@@
+			)
+		)
+		(property "MPN" "C6187"
+			(at 157.48 85.09 0)
+			(effects
+				(font
+					(size 1.27 1.27)
+				)
+				(hide yes)
 			)
 		)
@@
 			)
 		)
+		(property "MPN" "C13585"
+			(at 124.46 93.98 90)
+			(effects
+				(font
+					(size 1.27 1.27)
+				)
+				(hide yes)
+			)
+		)
 		(pin "2"
 		)
@@
 		(property "Description" "CL31A106KBHNNNE"
 			(at 167.64 93.98 0)
+			(effects
+				(font
+					(size 1.27 1.27)
+				)
+				(hide yes)
+			)
+		)
+		(property "MPN" "C13585"
+			(at 167.64 93.98 90)
 			(effects
 				(font
@@
 			)
 		)
+		(property "MPN" "C13585"
+			(at 104.14 93.98 90)
+			(effects
+				(font
+					(size 1.27 1.27)
+				)
+				(hide yes)
+			)
+		)
 		(pin "2"
 		)
@@
 			)
 		)
+		(property "MPN" "C6186"
+			(at 114.3 85.09 0)
+			(effects
+				(font
+					(size 1.27 1.27)
+				)
+				(hide yes)
+			)
+		)
 		(pin "2"
 		)
@@
 			(effects
 				(font
+					(size 1.27 1.27)
+				)
+				(hide yes)
+			)
+		)
+		(property "MPN" "C13585"
+			(at 147.32 93.98 90)
+			(effects
+				(font
