File: usbuart.kicad_sch (KiCad schematic)
At the start: 21 parts, among them J3 USB4056-03-A_REVA2, U10 FT231XQ-T, U7 CPDQ5V0-HF, U8 CPDQ5V0-HF, U9 CPDQ5V0-HF

Commit message: meant to put these in the last commit
Connections:
- net USB_D+ renamed USB_Internal_D+
- net USB_D- renamed USB_Internal_D-
Other:
- note added: "exposed for the header"
Changed lines of the file:
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@@
+		)
+	)
+	(text "exposed for the header"
+		(exclude_from_sim no)
+		(at 132.842 41.148 0)
+		(effects
+			(font
+				(size 0.889 0.889)
+			)
 		)
 	)
@@
 	)
 	(junction
-		(at 127 127)
-		(diameter 0)
-		(color 0 0 0 0)
-	)
-	(junction
 		(at 210.82 52.07)
 		(diameter 0)
@@
 	)
 	(junction
+		(at 142.24 86.36)
+		(diameter 0)
+		(color 0 0 0 0)
+	)
+	(junction
 		(at 62.23 93.98)
 		(diameter 0)
@@
 	(junction
 		(at 109.22 113.03)
+		(diameter 0)
+		(color 0 0 0 0)
+	)
+	(junction
+		(at 144.78 83.82)
 		(diameter 0)
 		(color 0 0 0 0)
@@
 	(wire
 		(pts
-			(xy 124.46 86.36) (xy 147.32 86.36)
+			(xy 124.46 86.36) (xy 142.24 86.36)
 		)
 		(stroke
@@
 	(wire
 		(pts
+			(xy 134.62 44.45) (xy 144.78 44.45)
+		)
+		(stroke
+			(width 0)
+			(type default)
+		)
+	)
+	(wire
+		(pts
 			(xy 69.85 76.2) (xy 73.66 76.2)
 		)
@@
 	(wire
 		(pts
+			(xy 142.24 46.99) (xy 142.24 86.36)
+		)
+		(stroke
+			(width 0)
+			(type default)
+		)
+	)
+	(wire
+		(pts
 			(xy 54.61 101.6) (xy 62.23 101.6)
 		)
@@
 	(wire
 		(pts
+			(xy 144.78 44.45) (xy 144.78 83.82)
+		)
+		(stroke
+			(width 0)
+			(type default)
+		)
+	)
+	(wire
+		(pts
 			(xy 207.01 87.63) (xy 208.28 87.63)
 		)
@@
 	(wire
 		(pts
+			(xy 144.78 83.82) (xy 147.32 83.82)
+		)
+		(stroke
+			(width 0)
+			(type default)
+		)
+	)
+	(wire
+		(pts
 			(xy 166.37 67.31) (xy 166.37 86.36)
 		)
@@
 	(wire
 		(pts
-			(xy 127 127) (xy 127 124.46)
-		)
-		(stroke
-			(width 0)
-			(type default)
-		)
-	)
-	(wire
-		(pts
 			(xy 171.45 54.61) (xy 167.64 54.61)
 		)
@@
 	(wire
 		(pts
-			(xy 127 132.08) (xy 127 127)
+			(xy 127 124.46) (xy 127 132.08)
 		)
 		(stroke
@@
 	(wire
 		(pts
+			(xy 142.24 86.36) (xy 147.32 86.36)
+		)
+		(stroke
+			(width 0)
+			(type default)
+		)
+	)
+	(wire
+		(pts
+			(xy 134.62 46.99) (xy 142.24 46.99)
+		)
+		(stroke
+			(width 0)
+			(type default)
+		)
+	)
+	(wire
+		(pts
 			(xy 54.61 93.98) (xy 62.23 93.98)
 		)
@@
 	(wire
 		(pts
-			(xy 132.08 114.3) (xy 132.08 127)
-		)
-		(stroke
-			(width 0)
-			(type default)
-		)
-	)
-	(wire
-		(pts
 			(xy 166.37 97.79) (xy 220.98 97.79)
 		)
@@
 	(wire
 		(pts
-			(xy 124.46 83.82) (xy 147.32 83.82)
+			(xy 124.46 83.82) (xy 144.78 83.82)
 		)
 		(stroke
@@
 		(pts
 			(xy 207.01 64.77) (xy 220.98 64.77)
-		)
-		(stroke
-			(width 0)
-			(type default)
-		)
-	)
-	(wire
-		(pts
-			(xy 132.08 127) (xy 127 127)
 		)
 		(stroke
@@
 	)
 	(label "USB_D-"
-		(at 147.32 86.36 180)
+		(at 140.97 86.36 180)
 		(effects
 			(font
@@
 	)
 	(label "USB_D+"
-		(at 147.32 83.82 180)
+		(at 140.97 83.82 180)
 		(effects
 			(font
@@
 		)
 	)
+	(hierarchical_label "USB_Internal_D+"
+		(shape passive)
+		(at 134.62 44.45 180)
+		(effects
+			(font
+				(size 1.27 1.27)
+			)
+			(justify right)
+		)
+	)
+	(hierarchical_label "USB_Internal_D-"
+		(shape passive)
+		(at 134.62 46.99 180)
+		(effects
+			(font
+				(size 1.27 1.27)
+			)
+			(justify right)
+		)
+	)
+	(hierarchical_label "DCD#"
+		(shape passive)
+		(at 118.11 125.73 0)
+		(effects
+			(font
+				(size 1.27 1.27)
+			)
+			(justify left)
+		)
+	)
 	(hierarchical_label "CTS#"
 		(shape input)
-		(at 132.08 114.3 90)
+		(at 127 125.73 0)
 		(effects
 			(font
@@
 		)
 	)
+	(hierarchical_label "DSR#"
+		(shape passive)
+		(at 109.22 125.73 0)
+		(effects
+			(font
+				(size 1.27 1.27)
+			)
+			(justify left)
+		)
+	)
 	(hierarchical_label "PowerOut"
 		(shape output)
@@
 		)
 	)
+	(hierarchical_label "RI#"
+		(shape passive)
+		(at 99.06 125.73 0)
+		(effects
+			(font
+				(size 1.27 1.27)
+			)
+			(justify left)
+		)
+	)

Commit message: designated MPN parts from JLC library
Parts:
- C11: MPN (none) -> C1779
- C17, C19: MPN (none) -> C1525
- D1, D2: MPN (none) -> C2286
- FB1: MPN (none) -> C1002
- J3: MPN (none) -> C7407280
- R10, R9: MPN (none) -> C23186
- R11, R12: MPN (none) -> C22966
- R13, R14: MPN (none) -> C23345
- R17, R18, R19, R20: MPN (none) -> C25804
- U10: MPN (none) -> C1521552
- U7, U8, U9: MPN (none) -> C2441615
Changed lines of the file:
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@@
+			)
+		)
+		(property "MPN" "C2441615"
+			(at 245.11 67.31 90)
+			(effects
+				(font
+					(size 1.27 1.27)
+				)
+				(hide yes)
 			)
 		)
@@
 			)
 		)
+		(property "MPN" "C25804"
+			(at 109.22 120.65 90)
+			(effects
+				(font
+					(size 1.27 1.27)
+				)
+				(hide yes)
+			)
+		)
 		(pin "2"
 		)
@@
 			)
 		)
+		(property "MPN" "C2441615"
+			(at 229.87 67.31 90)
+			(effects
+				(font
+					(size 1.27 1.27)
+				)
+				(hide yes)
+			)
+		)
 		(pin "2"
 		)
@@
 		)
 		(property "Sim.Pins" "1=K 2=A"
+			(at 71.12 129.54 0)
+			(effects
+				(font
+					(size 1.27 1.27)
+				)
+				(hide yes)
+			)
+		)
+		(property "MPN" "C2286"
 			(at 71.12 129.54 0)
 			(effects
@@
 			)
 		)
+		(property "MPN" "C1521552"
+			(at 124.46 66.04 0)
+			(effects
+				(font
+					(size 1.27 1.27)
+				)
+				(hide yes)
+			)
+		)
 		(pin "8"
 		)
@@
 			)
 		)
+		(property "MPN" "C25804"
+			(at 118.11 120.65 90)
+			(effects
+				(font
+					(size 1.27 1.27)
+				)
+				(hide yes)
+			)
+		)
 		(pin "2"
 		)
@@
 		)
 		(property "Sim.Pins" "1=K 2=A"
+			(at 81.28 129.54 0)
+			(effects
+				(font
+					(size 1.27 1.27)
+				)
+				(hide yes)
+			)
+		)
+		(property "MPN" "C2286"
 			(at 81.28 129.54 0)
 			(effects
@@
 			)
 		)
+		(property "MPN" "C23186"
+			(at 213.36 74.93 0)
+			(effects
+				(font
+					(size 1.27 1.27)
+				)
+				(hide yes)
+			)
+		)
 		(pin "2"
 		)
@@
 		(property "Description" "0603WAF2700T5E"
 			(at 81.28 118.11 0)
+			(effects
+				(font
+					(size 1.27 1.27)
+				)
+				(hide yes)
+			)
+		)
+		(property "MPN" "C22966"
+			(at 81.28 118.11 90)
 			(effects
 				(font
@@
 			)
 		)
+		(property "MPN" "C1779"
+			(at 54.61 101.6 90)
+			(effects
+				(font
+					(size 1.27 1.27)
+				)
+				(hide yes)
+			)
+		)
 		(pin "1"
 		)
@@
 		(property "Description" "0603WAF1002T5E"
 			(at 99.06 120.65 0)
+			(effects
+				(font
+					(size 1.27 1.27)
+				)
+				(hide yes)
+			)
+		)
+		(property "MPN" "C25804"
+			(at 99.06 120.65 90)
 			(effects
 				(font
@@
 			)
 		)
+		(property "MPN" "C23186"
+			(at 156.21 68.58 0)
+			(effects
+				(font
+					(size 1.27 1.27)
+				)
+				(hide yes)
+			)
+		)
 		(pin "2"
 		)
@@
 			)
 		)
+		(property "MPN" "C1525"
+			(at 62.23 101.6 90)
+			(effects
+				(font
+					(size 1.27 1.27)
+				)
+				(hide yes)
+			)
+		)
 		(pin "2"
 		)
@@
 			)
 		)
+		(property "MPN" "C1002"
+			(at 213.36 88.9 90)
+			(effects
+				(font
+					(size 1.27 1.27)
+				)
+				(hide yes)
+			)
+		)
 		(pin "2"
 		)
@@
 		(property "Description" ""
 			(at 237.49 67.31 0)
+			(effects
+				(font
+					(size 1.27 1.27)
+				)
+				(hide yes)
+			)
+		)
+		(property "MPN" "C2441615"
+			(at 237.49 67.31 90)
 			(effects
 				(font
@@
 			)
 		)
+		(property "MPN" "C23345"
+			(at 151.13 86.36 90)
+			(effects
+				(font
+					(size 1.27 1.27)
+				)
+				(hide yes)
+			)
+		)
 		(pin "2"
 		)
@@
 			)
 		)
+		(property "MPN" "C7407280"
+			(at 189.23 64.77 0)
+			(effects
+				(font
+					(size 1.27 1.27)
+				)
+				(hide yes)
+			)
+		)
 		(pin "B4"
 		)
@@
 		(property "Description" "CL05B104KO5NNNC"
 			(at 125.73 97.79 0)
+			(effects
+				(font
+					(size 1.27 1.27)
+				)
+				(hide yes)
+			)
+		)
+		(property "MPN" "C1525"
+			(at 125.73 97.79 90)
 			(effects
 				(font
@@
 			)
 		)
+		(property "MPN" "C23345"
+			(at 151.13 83.82 90)
+			(effects
+				(font
+					(size 1.27 1.27)
+				)
+				(hide yes)
+			)
+		)
 		(pin "2"
 		)
@@
 			)
 		)
+		(property "MPN" "C25804"
+			(at 127 120.65 90)
+			(effects
+				(font
+					(size 1.27 1.27)
+				)
+				(hide yes)
+			)
+		)
 		(pin "2"
 		)
@@
 			(effects
 				(font
+					(size 1.27 1.27)
+				)
+				(hide yes)
+			)
+		)
+		(property "MPN" "C22966"
+			(at 71.12 118.11 90)
+			(effects
+				(font

Commit message: Updated part numbers
Parts:
- removed FB1: GZ1608D601TF, Inductor_SMD:L_Sunlord_MWSA0603S, symbol Device:FerriteBead
- D1: value RX_STATUS_LED -> LED
- D2: value TX_STATUS_LED -> LED
- J3: footprint USB4056_03_A:GCT_USB4056-03-A_REVA2 -> 12402012E212A_AMP; symbol USB4056_03_A:USB4056-03-A_REVA2 -> 12402012E212A:12402012E212A; FIX (none) -> 1; MPN C7407280 -> C2765186
Connections:
- net GND: now also J3.A1-B12 (GND), J3.B1-A12 (GND); no longer J3.A1 (GND_A), J3.A12 (GND_A__1), J3.B1 (GND_B), J3.B12 (GND_B__1)
- net PowerOut: now also J3.A4-B9 (VBUS), J3.B4-A9 (VBUS); no longer J3.A4 (VBUS_A), J3.A9 (VBUS_A__1), J3.B4 (VBUS_B), J3.B9 (VBUS_B__1)
- no-connect marks 12 -> 4
Other:
- moved on the sheet: R9, U7, U8, U9
